File: pcb/NomadLeft/Nomad.sch (KiCad schematic (older format))
At the start: 64 parts, among them J1 AudioJack4, SW0:0 SW_Push, SW0:1 SW_Push, SW0:2 SW_Push, SW0:3 SW_Push, SW0:5 SW_Push, SW1:1 SW_Push, SW1:2 SW_Push, SW1:3 SW_Push, SW1:4 SW_Push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

Commit message: Fix schematics by rescuing symbols.
Parts:
- U1: symbol teensy:Teensy2.0_(C) -> Nomad-rescue:Teensy2.0_(C)-teensy
Changed lines of the file:
@@
 $EndDescr
 $Comp
-L teensy:Teensy2.0_(C) U1
+L Nomad-rescue:Teensy2.0_(C)-teensy U1
 U 1 1 5D9E787D
 P 4150 6800
